File: 7segment/7segment.kicad_pcb (KiCad board)
At the start: 2 copper layers, 147.3 x 96.5 mm, 33 parts, among them J1 Barrel_Jack, J2 Conn_Segments, J3 Conn_Segments, J4 Conn_Segments, J5 DB9_Male, SW1 SW_Push, SW2 SW_Push, U1 ULN2803A, U2 2981, U3 2981, U4 L7809, U5 74HC595, U6 74HC595, U7 4017, U8 StepUp, U9 Max3232Board

Commit message: KiCad: Platinen Version 1
Parts:
- removed R7: 10k, Resistor_THT:R_Axial_DIN0309_L9.0mm_D3.2mm_P12.70mm_Horizontal
- removed R8, R9: 10k, Resistor_THT:R_Axial_DIN0204_L3.6mm_D1.6mm_P7.62mm_Horizontal
- removed SW1, SW2: SW_Push, Button_Switch_THT:SW_PUSH_6mm_H7.3mm
- removed U8: StepUp, 7segment:StepUp
- added C10: 100nF, Capacitor_THT:C_Disc_D5.0mm_W2.5mm_P2.50mm, F.Cu at (263.3, 145.7)
- added C5: 100nF, Capacitor_THT:C_Disc_D5.0mm_W2.5mm_P2.50mm, F.Cu at (248.3, 143.5)
- added C6: 0,1uF, Capacitor_THT:C_Disc_D3.4mm_W2.1mm_P2.50mm, F.Cu at (205.7, 106.7)
- added C7: 1000uF, Capacitor_THT:CP_Radial_D10.0mm_P5.00mm, F.Cu at (224.2, 140.3)
- added C8: 100nF, Capacitor_THT:C_Disc_D5.0mm_W2.5mm_P2.50mm, F.Cu at (262.9, 89.4)
- added C9: 100nF, Capacitor_THT:C_Disc_D5.0mm_W2.5mm_P2.50mm, F.Cu at (264.4, 117.7)
- added D2: D, Diode_THT:D_A-405_P7.62mm_Horizontal, F.Cu at (205.7, 120.7)
- added F1: Fuse, myself:Fuse, F.Cu at (210.8, 90.2)
- added J6: Conn_01x03, myself:Connector 3xPin, F.Cu at (232.4, 59.7)
- added J7: Conn_01x03, myself:Connector 3xPin, F.Cu at (201.9, 59.7)
- added J8: Conn_01x03, myself:Connector 3xPin, F.Cu at (217.2, 59.7)
- C1: value CP -> 330uF; footprint Capacitor_THT:CP_Radial_D5.0mm_P2.50mm -> Capacitor_THT:CP_Radial_D10.0mm_P5.00mm
- C2: value CP -> 0,1uF; footprint Capacitor_THT:CP_Radial_D5.0mm_P2.50mm -> Capacitor_THT:C_Disc_D3.4mm_W2.1mm_P2.50mm
- C3, C4: footprint Capacitor_THT:CP_Radial_D5.0mm_P2.50mm -> Capacitor_THT:C_Disc_D5.0mm_W2.5mm_P2.50mm
- D1: footprint Diode_THT:D_A-405_P5.08mm_Vertical_KathodeUp -> Diode_THT:D_A-405_P10.16mm_Horizontal
- J1: value Barrel_Jack -> Conn_01x02; footprint Connector_PinHeader_2.54mm:PinHeader_1x02_P2.54mm_Vertical -> myself:Connector 2xPin
- J5: value DB9_Male -> Conn_01x03; footprint Connector_Dsub:DSUB-9_Male_Vertical_P2.77x2.84mm -> myself:Connector 3xPin
- R1: value R -> 100k; footprint Resistor_THT:R_Axial_DIN0204_L3.6mm_D1.6mm_P7.62mm_Horizontal -> myself:Resistor, L6mm,4holes
- R10, R3: footprint Resistor_THT:R_Axial_DIN0204_L3.6mm_D1.6mm_P7.62mm_Horizontal -> myself:Resistor, L6mm,4holes
- R11, R4: footprint Resistor_THT:R_Axial_DIN0204_L3.6mm_D1.6mm_P7.62mm_Horizontal -> myself:Resistor, L6mm,5holes
- R2: value R -> 10k; footprint Resistor_THT:R_Axial_DIN0207_L6.3mm_D2.5mm_P10.16mm_Horizontal -> myself:Resistor, L6mm,5holes
- R5: footprint Resistor_THT:R_Axial_DIN0207_L6.3mm_D2.5mm_P10.16mm_Horizontal -> myself:Resistor, L6mm,6holes
- R6: footprint Resistor_THT:R_Axial_DIN0207_L6.3mm_D2.5mm_P10.16mm_Horizontal -> myself:Resistor, L6mm,5holes
- U1: footprint Package_DIP:DIP-18_W7.62mm -> Package_DIP:DIP-18_W7.62mm_LongPads
- U4: value L7809 -> L7805; footprint Connector_PinSocket_2.54mm:PinSocket_1x03_P2.54mm_Vertical -> L7805CV:TO255P1040X460X1968-3
- U5, U6, U7: footprint Package_DIP:DIP-16_W7.62mm -> Package_DIP:DIP-16_W7.62mm_LongPads
- U9: footprint 7segment:MAX232 -> myself:MAX232
- moved J5 185.3 mm to (204.5, 134.0), turned to 90 degrees
- moved C4 54.6 mm to (248.3, 113.0), turned to 180 degrees
- moved R4 46.2 mm to (222.2, 106.7), turned to 90 degrees
- moved R5 45.9 mm to (227.3, 106.7), turned to 90 degrees
- moved J1 42.3 mm to (196.8, 76.2), turned to 90 degrees
- moved R2 39.9 mm to (224.8, 111.8)
- moved C1 37.5 mm to (204.5, 88.9), turned to 180 degrees
- moved R1 32.2 mm to (214.6, 109.2)
- moved C3 29.9 mm to (248.3, 85.1), turned to 180 degrees
- moved A1 29.7 mm to (233.7, 119.4)
- moved C2 27.9 mm to (205.7, 97.8), turned to 180 degrees
- moved U9 27.3 mm to (224.8, 129.5)
- moved D1 26.8 mm to (201.3, 110.5), turned to 0 degrees
- moved R6 21.1 mm to (238.1, 76.2), turned to 270 degrees
- moved R3 19.7 mm to (229.9, 106.7)
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Connections:
- A1 pad 1: Tx -> Net-(A1-Pad1)
- A1 pad 10: Net-(A1-Pad10) -> ArduinoD7
- A1 pad 11: Net-(A1-Pad11) -> (no net)
- A1 pad 14: ArduinoD11 -> Net-(A1-Pad14)
- A1 pad 15: ArduinoD12 -> Net-(A1-Pad15)
- A1 pad 16: Net-(A1-Pad16) -> (no net)
- A1 pad 17: Net-(A1-Pad17) -> (no net)
- A1 pad 18: Net-(A1-Pad18) -> (no net)
- A1 pad 19: Net-(A1-Pad19) -> (no net)
- A1 pad 2: Rx -> Net-(A1-Pad2)
- A1 pad 22: Net-(A1-Pad22) -> (no net)
- A1 pad 23: Net-(A1-Pad23) -> (no net)
- A1 pad 24: Net-(A1-Pad24) -> (no net)
- A1 pad 26: Net-(A1-Pad26) -> (no net)
- A1 pad 28: Net-(A1-Pad28) -> (no net)
- A1 pad 3: Net-(A1-Pad3) -> (no net)
- A1 pad 30: +9V -> (no net)
- C1 pad 1: Net-(C1-Pad1) -> +15V
- C2 pad 1: +9V -> GND
- C2 pad 2: GND -> +15V
- C3 pad 1: ArduinoD11 -> GND
- C3 pad 2: GND -> +5V
- C4 pad 1: ArduinoD12 -> GND
- C4 pad 2: GND -> +5V
- D1 pad 1: Net-(C1-Pad1) -> +15V
- D1 pad 2: +9V -> +5V
- J1 pad 1: Net-(C1-Pad1) -> Net-(F1-Pad2)
- J5 pad 3: Net-(J5-Pad3) -> GND
- R1 pad 1: Net-(C1-Pad1) -> +15V
- R4 pad 1: GND -> +5V
- R6 pad 1: ArduinoD11 -> GND
- R6 pad 2: Net-(R6-Pad2) -> ArduinoD7
- U2 pad 9: +24V -> +15V
- U3 pad 9: +24V -> +15V
- U4 pad 1: Net-(C1-Pad1) -> +15V
- U4 pad 3: +9V -> +5V
- U5 pad 11: ArduinoD5 -> ArduinoD7
- U5 pad 13: GND -> ArduinoD5
- U5 pad 9: Net-(U5-Pad9) -> (no net)
- U6 pad 11: ArduinoD5 -> ArduinoD7
- U6 pad 13: GND -> ArduinoD5
- U7 pad 11: Net-(U7-Pad11) -> (no net)
- U7 pad 12: Net-(U7-Pad12) -> (no net)
- U7 pad 9: Net-(U7-Pad9) -> (no net)
- U9 pad 0: Net-(J5-Pad3) -> Net-(J5-Pad2)
- U9 pad 1: Net-(J5-Pad2) -> Net-(J5-Pad1)
- U9 pad 2: Tx -> Net-(A1-Pad2)
- U9 pad 3: Rx -> Net-(A1-Pad1)
Routing:
- net +15V: track 0.00 -> 226.3 mm, vias 0 -> 2
- net +24V: track 135.1 -> 0.00 mm, vias 5 -> 0
- net (no net): track 0.00 -> 114.3 mm
- net GND: track 478.7 -> 417.9 mm, vias 23 -> 2
- net +5V: track 219.5 -> 274.9 mm, vias 11 -> 10
- net +9V: track 48.3 -> 0.00 mm, vias 2 -> 0
- net ArduinoD7: track 0.00 -> 46.2 mm
- net Net-(A1-Pad20): track 0.00 -> 41.4 mm
- net Net-(A1-Pad21): track 0.00 -> 40.4 mm
- net ArduinoD2: track 73.7 -> 35.2 mm, vias 4 -> 0
- net ArduinoD3: track 73.7 -> 36.7 mm, vias 4 -> 0
- net Net-(A1-Pad12): track 0.00 -> 33.2 mm
- net Net-(U1-Pad1): track 47.2 -> 16.8 mm, vias 4 -> 2
- net Net-(A1-Pad13): track 0.00 -> 28.6 mm
- net ArduinoD4: track 43.2 -> 15.9 mm, vias 2 -> 0
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- added copper zone on B.Cu, net (none)
- added copper zone on B.Cu, net GND
Other:
- board size 147.3 x 96.5 mm -> 91.4 x 99.1 mm
- net class 15V added: clearance 0.4, trace_width 1, via_dia 2, via_drill 0.8
- net class Default: clearance 0.2 -> 0.4; trace_width 0.25 -> 0.5; via_dia 0.8 -> 2; via_drill 0.4 -> 0.8
- rule trace_clearance: 0.2 -> 0.4
- board text added: "15V"
- board text added: "99 mm"
- board text added: "B1 B2 GND"
- board text added: "GND"
- board text added: "RS232 Pin2 Pin3 Pin9"
